File: as7265x_color_sensors/as7265x_color_sensors.sch (KiCad schematic (older format))
At the start: 3 parts

Commit message: added basic sensor chips with led outputs
Parts:
- added C? (x3): 100nF, symbol Device:C_Small
- added C? (x3): 10uF, symbol Device:C_Small
- added D? (x6): LED_Small, symbol Device:LED_Small
- added J?: Conn_01x06_Male, symbol Connector:Conn_01x06_Male
- added R?: 10k, symbol Device:R_Small
- added R? (x6): R_Small, symbol Device:R_Small
- added TP? (x2): TestPoint, symbol Connector:TestPoint
Connections:
- net labels added: 3V3, CTS, DTR, GND, LED1, LED2, LED3, LED4, LED5, LED6, RXI, TXO, ~INT
- wire segments 0 -> 84
- no-connect marks 0 -> 6
Other:
- note added: "Connector for SparkFun FTDI Basic Breakout - 3.3V"

Commit message: schematic almost done, missing some footprints for the color sensors, place holders used
Parts:
- added C7: 1uF, Capacitor_SMD:C_0805_2012Metric, symbol Device:C_Small
- added F1, F2: Polyfuse, Capacitor_SMD:C_1206_3216Metric, symbol Device:Polyfuse
- added J2, J3: RJ12, Connector_RJ:RJ12_Amphenol_54601, symbol Connector:RJ12
- added R10, R11, R12, R13: 10K, Resistor_SMD:R_0805_2012Metric, symbol Device:R_Small
- added R8: DNP, Resistor_SMD:R_0805_2012Metric, symbol Device:R_Small
- added R9: 0R, Resistor_SMD:R_0805_2012Metric, symbol Device:R_Small
- added U4: AT25SF041, Package_DIP:DIP-8_W7.62mm, symbol Memory_EEPROM:AT25xxx
- C1: renamed from C?; footprint (none) -> Capacitor_SMD:C_1206_3216Metric
- C2, C3, C4, C5, C6: renamed from C?; footprint (none) -> Capacitor_SMD:C_0805_2012Metric
- D1, D2, D3, D4, D5, D6: renamed from D?; footprint (none) -> LED_SMD:LED_1206_3216Metric
- J1: renamed from J?; footprint (none) -> Connector_Harwin:Harwin_M20-89006xx_1x06_P2.54mm_Horizontal
- R1, R2, R3, R4, R5, R6, R7: renamed from R?; footprint (none) -> Resistor_SMD:R_0805_2012Metric
- TP1, TP2: renamed from TP?; footprint (none) -> Connector_Pin:Pin_D1.0mm_L10.0mm_LooseFit
- U1, U2, U3: renamed from U?; footprint (none) -> Package_DFN_QFN:ST_UFQFPN-20_3x3mm_P0.5mm
Connections:
- wire segments 84 -> 155
- no-connect marks 6 -> 15

Commit message: chip footprints fixed, started layout
Parts:
- C1: footprint Capacitor_SMD:C_1206_3216Metric -> Capacitor_SMD:C_0805_2012Metric
- U1: renamed from U3; footprint Package_DFN_QFN:ST_UFQFPN-20_3x3mm_P0.5mm -> MRV_SMD_Packages:LGA-20_4.5mm_4.7mm_2.5mm
- U2: renamed from U1; footprint Package_DFN_QFN:ST_UFQFPN-20_3x3mm_P0.5mm -> MRV_SMD_Packages:LGA-20_4.5mm_4.7mm_2.5mm
- U3: renamed from U2; footprint Package_DFN_QFN:ST_UFQFPN-20_3x3mm_P0.5mm -> MRV_SMD_Packages:LGA-20_4.5mm_4.7mm_2.5mm
- U4: footprint Package_DIP:DIP-8_W7.62mm -> Package_SO:SOIC-8_3.9x4.9mm_P1.27mm
Changed lines of the file:
@@
 $EndDescr
 $Comp
-L MRV_ICs:AS72651 U3
+L MRV_ICs:AS72651 U1
 U 1 1 5B67836C
 P 3050 2550
-F 0 "U3" H 3300 2600 50  0000 C CNN
+F 0 "U1" H 3300 2600 50  0000 C CNN
 F 1 "AS72651" H 3650 2650 50  0000 C CNN
-F 2 "Package_DFN_QFN:ST_UFQFPN-20_3x3mm_P0.5mm" H 3050 2550 50  0001 C CNN
+F 2 "MRV_SMD_Packages:LGA-20_4.5mm_4.7mm_2.5mm" H 3050 2550 50  0001 C CNN
 F 3 "" H 3050 2550 50  0001 C CNN
 	1    3050 2550
@@
 $EndComp
 $Comp
-L MRV_ICs:AS72652 U1
+L MRV_ICs:AS72652 U2
 U 1 1 5B67842B
 P 3000 4400
-F 0 "U1" H 3300 4500 50  0000 C CNN
+F 0 "U2" H 3300 4500 50  0000 C CNN
 F 1 "AS72652" H 3700 4600 50  0000 C CNN
-F 2 "Package_DFN_QFN:ST_UFQFPN-20_3x3mm_P0.5mm" H 4300 4550 50  0001 C CNN
+F 2 "MRV_SMD_Packages:LGA-20_4.5mm_4.7mm_2.5mm" H 4300 4550 50  0001 C CNN
 F 3 "" H 4300 4550 50  0001 C CNN
 	1    3000 4400
@@
 $EndComp
 $Comp
-L MRV_ICs:AS72653 U2
+L MRV_ICs:AS72653 U3
 U 1 1 5B6785AF
 P 3000 6100
-F 0 "U2" H 3250 6200 50  0000 C CNN
+F 0 "U3" H 3250 6200 50  0000 C CNN
 F 1 "AS72653" H 3700 6250 50  0000 C CNN
-F 2 "Package_DFN_QFN:ST_UFQFPN-20_3x3mm_P0.5mm" H 3150 5800 50  0001 C CNN
+F 2 "MRV_SMD_Packages:LGA-20_4.5mm_4.7mm_2.5mm" H 3150 5800 50  0001 C CNN
 F 3 "" H 3150 5800 50  0001 C CNN
 	1    3000 6100
@@
 F 0 "C1" H 1600 1450 50  0000 L CNN
 F 1 "100nF" H 1500 1350 50  0000 L CNN
-F 2 "Capacitor_SMD:C_1206_3216Metric" H 1800 1400 50  0001 C CNN
+F 2 "Capacitor_SMD:C_0805_2012Metric" H 1800 1400 50  0001 C CNN
 F 3 "~" H 1800 1400 50  0001 C CNN
 	1    1800 1400
@@
 F 0 "U4" H 5700 1650 50  0000 C CNN
 F 1 "AT25SF041" H 5300 1150 50  0000 C CNN
-F 2 "Package_DIP:DIP-8_W7.62mm" H 5600 1400 50  0001 C CNN
+F 2 "Package_SO:SOIC-8_3.9x4.9mm_P1.27mm" H 5600 1400 50  0001 C CNN
 F 3 "http://ww1.microchip.com/downloads/en/DeviceDoc/Atmel-8707-SEEPROM-AT25010B-020B-040B-Datasheet.pdf" H 5600 1400 50  0001 C CNN
 	1    5600 1400

Commit message: added more info to schematic
Other:
- note added: "Comm port"
- note added: "Expansion Color Sensor"
- note added: "FTDI Plug"
- note added: "Firmware"
- note added: "LED port\n"
- note added: "Master Color Sensor"
Changed lines of the file:
@@
 Wire Wire Line
 	9400 3450 9650 3450
+Text Notes 7400 4600 0    157  ~ 0
+LED port\n
+Text Notes 7250 3750 0    157  ~ 0
+Comm port
+Text Notes 6500 1550 0    157  ~ 0
+Firmware
+Text Notes 2150 1050 0    157  ~ 0
+Master Color Sensor
+Text Notes 4650 4100 0    157  ~ 0
+Expansion Color Sensor
+Text Notes 4650 5900 0    157  ~ 0
+Expansion Color Sensor
+Text Notes 7250 5700 0    157  ~ 0
+FTDI Plug
 $EndSCHEMATC

Commit message: adding TVS diode arrays
Parts:
- added TVS1, TVS2, TVS3: SP3012-06UTG, MRV_SMD_Packages:uDFN-14_3.5x1.35x0.5mm, symbol MRV_Passives:SP3012-06UTG
Connections:
- wire segments 155 -> 184
Other:
- note added: "SP3012-06UTG for protection"
- moved on the sheet: J2, J3

Commit message: added test points, more layout progress
Parts:
- added TP10, TP11, TP12, TP13, TP14, TP15, TP16, TP17, TP3, TP4, TP5, TP6, TP7, TP8, TP9: TestPoint, Connector_Pin:Pin_D1.0mm_L10.0mm_LooseFit, symbol Connector:TestPoint
Connections:
- wire segments 184 -> 202
- no-connect marks 15 -> 14
Other:
- note removed: "SP3012-06UTG for protection"

Commit message: layout looks just about done
Parts:
- removed TP16, TP7: TestPoint, Connector_Pin:Pin_D1.0mm_L10.0mm_LooseFit, symbol Connector:TestPoint
Changed lines of the file:
@@
 	10200 5850 10850 5850
-$Comp
-L Connector:TestPoint TP7
-U 1 1 5B698AD5
-P 5800 5300
-F 0 "TP7" H 5750 5500 50  0000 L CNN
-F 1 "TestPoint" H 5858 5329 50  0001 L CNN
-F 2 "Connector_Pin:Pin_D1.0mm_L10.0mm_LooseFit" H 6000 5300 50  0001 C CNN
-F 3 "~" H 6000 5300 50  0001 C CNN
-	1    5800 5300
-	1    0    0    -1
-$EndComp
 $Comp
 L Connector:TestPoint TP10
@@
 	1    0    0    -1
 $EndComp
-$Comp
-L Connector:TestPoint TP16
-U 1 1 5B71C6CC
-P 10400 5800
-F 0 "TP16" H 10200 6000 50  0000 L CNN
-F 1 "TestPoint" H 10458 5829 50  0001 L CNN
-F 2 "Connector_Pin:Pin_D1.0mm_L10.0mm_LooseFit" H 10600 5800 50  0001 C CNN
-F 3 "~" H 10600 5800 50  0001 C CNN
-	1    10400 5800
-	1    0    0    -1
-$EndComp
